File: PCB/ProvisioningJig_v3.1/ProvisioningJig_v3.kicad_pcb (KiCad board)
At the start: 2 copper layers, 85 x 56 mm, 52 parts, among them J2 Raspberry_Pi_2_3, J3 POGO USB1+, J4 POGO USB1-, J6 POGO USB2+, J7 POGO USB2-, Q1 S8050_SMD, Q2 AO3401A, Q3 S8050_SMD, Q4 S8050_SMD, Q5 S8050_SMD, Q6 AO3401A, Q7 S8050_SMD, Q8 AO3401A, Q9 S8050_SMD, U1 New Version Debugger, U2 ST-Link, U3 Target, U5 LM393

Commit message: fixed target slot
Routing:
- net /D_SWCLK: track 102.2 -> 104.8 mm
- net /Target_PWR: track 172.1 -> 173.6 mm
- net /D_SWIO: track 139.1 -> 140.5 mm
- net GND: track 249.6 -> 250.6 mm
